File: Electronics/Newbies.kicad_sch (KiCad schematic)
At the start: 14 parts, among them J1 USB_C_Receptacle_USB2.0_14P, U1 ESP32-S3-WROOM-1, U2 NCP1117-3.3_SOT223, U3 NCP1117-3.3_SOT223, U4 MOTOR_L

Commit message: Add Electronics KiCad project files (from attachment)
Parts:
- added C7, C8: 100u, symbol Device:C
- added R3, R4: R, symbol Device:R
- added U5: ~, symbol bmi270:BMI270
Connections:
- net +3V3: now also C7.2, C8.1, R3.1, R4.1, U5.5 (VDDIO), U5.8 (VDD)
- net GND: now also C7.1, C8.2, U5.6 (GNDIO), U5.7 (GND)
- net IMU_SDA: now reaches U1.18 (IO10)
- net IMU_SDA: now also R3.2, U5.14 (SDX)
- net IMU_SCL: now reaches U1.19 (IO11)
- net IMU_SCL: now also R4.2, U5.13 (SCX)

Commit message: Update Electronics KiCad schematic (Newbies.kicad_sch)
Parts:
- R3, R4: value R -> 2.2K
Connections:
- net IMU_SCL renamed SCL
- net IMU_SDA renamed SDA
Changed lines of the file:
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@@
 	(wire
 		(pts
-			(xy 163.83 190.5) (xy 168.91 190.5)
+			(xy 163.83 185.42) (xy 171.45 185.42)
 		)
 		(stroke
@@
 		(pts
 			(xy 139.7 181.61) (xy 139.7 186.69)
-		)
-		(stroke
-			(width 0)
-			(type default)
-		)
-	)
-	(wire
-		(pts
-			(xy 163.83 185.42) (xy 163.83 190.5)
 		)
 		(stroke
@@
 		)
 	)
-	(label "IMU_SDA"
+	(label "SDA"
 		(at 132.08 134.62 270)
 		(effects
@@
 		)
 	)
-	(label "IMU_SCL"
+	(label "SCL"
 		(at 144.78 109.22 180)
 		(effects
@@
 		)
 	)
-	(label "IMU_SCL"
+	(label "SCL"
 		(at 139.7 134.62 270)
 		(effects
@@
 		)
 	)
-	(label "IMU_SDA"
+	(label "SDA"
 		(at 144.78 106.68 180)
 		(effects
@@
 		(lib_name "+3V3_1")
 		(lib_id "power:+3V3")
-		(at 168.91 190.5 0)
+		(at 171.45 185.42 0)
 		(unit 1)
 		(exclude_from_sim no)
@@
 		(fields_autoplaced yes)
 		(property "Reference" "#PWR012"
-			(at 168.91 194.31 0)
+			(at 171.45 189.23 0)
 			(effects
 				(font
@@
 		)
 		(property "Value" "+3V3"
-			(at 168.91 185.42 0)
+			(at 171.45 180.34 0)
 			(effects
 				(font
@@
 		)
 		(property "Footprint" ""
-			(at 168.91 190.5 0)
+			(at 171.45 185.42 0)
 			(effects
 				(font
@@
 		)
 		(property "Datasheet" ""
-			(at 168.91 190.5 0)
+			(at 171.45 185.42 0)
 			(effects
 				(font
@@
 		)
 		(property "Description" "Power symbol creates a global label with name \"+3V3\""
-			(at 168.91 190.5 0)
+			(at 171.45 185.42 0)
 			(effects
 				(font
@@
 			)
 		)
-		(property "Value" "R"
+		(property "Value" "2.2K"
 			(at 113.03 170.1799 0)
 			(effects
@@
 			)
 		)
-		(property "Value" "R"
+		(property "Value" "2.2K"
 			(at 120.65 165.0999 0)
 			(effects

Commit message: johnny stuff
Parts:
- added C10: 0.1uf, symbol Device:C
- added C5: 100n, symbol Device:C
- added C9: 22n, symbol Device:C
- added J2, J3: Screw_Terminal_01x04, symbol Connector:Screw_Terminal_01x04
- added R10, R9: 330m, symbol Device:R
- added R11, R12, R5, R6, R7, R8: 10k, symbol Device:R
- added SW1, SW2, SW3, SW4, SW5, SW6: SW_Push, symbol Switch:SW_Push
- added U4: MOTOR_R, Package_DFN_QFN:QFN-28-1EP_5x5mm_P0.5mm_EP3.75x3.75mm, symbol TMC2209-LA-T:TMC2209-LA-T
Connections:
- net +3V3: now also C10.1, R11.1, R12.1, R5.1, R6.1, R7.1, R8.1, SW1.1, SW2.1, SW3.1, SW4.1, SW5.1, SW6.1, U4.15 (VCC_IO)
- net DIR_L: now also U1.9 (IO16)
- net GND: now also C10.2, R10.2, R5.2, R6.2, R7.2, R8.2, R9.2, SW1.2, SW2.2, U4.13 (CLK), U4.18 (GND), U4.29 (GND), U4.3 (GND)
- net LA1: now also J2.1 (Pin_1)
- net LA2: now also J2.2 (Pin_2)
- net LB1: now also J2.3 (Pin_3)
- net LB2: now also J2.4 (Pin_4)
- net STEP_L: now also U1.8 (IO15)
- net VBAT: now also C5.1, U4.22 (VS), U4.28 (VS)
- net VREF: now also U4.17 (VREF)
- net ~{EN}: now also U1.20 (IO12), U4.2 (ENN)
- net BTN3: now reaches U1.12 (IO8)
- net BTN3: now also SW5.2
- net BTN4: now reaches U1.17 (IO9)
- net BTN4: now also SW6.2
- net STEP_R: now reaches U1.21 (IO13)
- net STEP_R: now also U4.16 (STEP)
- net DIR_R: now reaches U1.22 (IO14)
- net DIR_R: now also U4.19 (DIR)
- net BOOT: now reaches U1.27 (IO0)
- net BOOT: now also R12.2
- net EN: now reaches U1.3 (EN)
- net EN: now also R11.2
- net BTN1: now reaches U1.6 (IO6)
- net BTN1: now also SW3.2
- net BTN2: now reaches U1.7 (IO7)
- net BTN2: now also SW4.2
- net AD0_L: no longer names the net of U4.9 (MS1_AD0)
- net AD1_L: no longer names the net of U4.10 (MS1_AD1)
- new net: C9.1, U4.4 (CPO)
- new net: C9.2, U4.5 (CPI)
- new net: C5.2, U4.6 (VCP)
- new net: R10.1, U4.27 (BRB)
- new net: R9.1, U4.23 (BRA)
- new net RA1: J3.1 (Pin_1), U4.24 (OA1)
- new net RA2: J3.2 (Pin_2), U4.21 (OA2)
- new net RB1: J3.3 (Pin_3), U4.26 (OB1)
- new net RB2: J3.4 (Pin_4), U4.1 (OB2)
- no-connect marks 8 -> 18
Other:
- moved on the sheet: C5, C6, R1, R2, U1
